Commit message: fix home position and add apple proxy

File: urdf/tables_v2.urdf.xacro (robot description, xacro)
@@ -71,32 +71,32 @@
       </collision>
     </link>
-<!--    <link name="apple_stem" >-->
-<!--      <visual>-->
-<!--        <origin xyz="0 0 0" rpy="0 0 0"/>-->
-<!--        <geometry>-->
-<!--          <mesh filename="package://millrace_moveit_config/meshes/millrace_moveit_config/visual/Stem_v4.STL" scale="0.001 0.001 0.001"/>-->
-<!--        </geometry>-->
-<!--        <material name="Orange">-->
-<!--          <color rgba="1 0.65 0 1.0"/>-->
-<!--        </material>-->
-<!--      </visual>-->
-<!--      <collision>-->
-<!--        <origin xyz="0 0 0" rpy="0 0 0"/>-->
-<!--        <geometry>-->
-<!--          <mesh filename="package://millrace_moveit_config/meshes/millrace_moveit_config/collision/Proxy_V1_collision.STL" scale="0.001 0.001 0.001"/>-->
-<!--        </geometry>-->
-<!--      </collision>-->
-<!--    </link>-->
-<!--    <link name="apple" >-->
-<!--      <visual>-->
-<!--        <origin xyz="0 0 0" rpy="0 0 0"/>-->
-<!--        <geometry>-->
-<!--          <mesh filename="package://millrace_moveit_config/meshes/millrace_moveit_config/visual/SubAssem_Apple_V4.STL" scale="0.001 0.001 0.001"/>-->
-<!--        </geometry>-->
-<!--        <material name="Red">-->
-<!--          <color rgba="1.0 0.0 0.0 1.0"/>-->
-<!--        </material>-->
-<!--      </visual>-->
-<!--    </link>-->
+    <link name="apple_stem" >
+      <visual>
+        <origin xyz="0 0 0" rpy="0 0 0"/>
+        <geometry>
+          <mesh filename="package://millrace_moveit_config/meshes/apple_proxy/visual/Stem_v4.STL" scale="0.001 0.001 0.001"/>
+        </geometry>
+        <material name="Orange">
+          <color rgba="1 0.65 0 1.0"/>
+        </material>
+      </visual>
+      <collision>
+        <origin xyz="0 0 0" rpy="0 0 0"/>
+        <geometry>
+          <mesh filename="package://millrace_moveit_config/meshes/apple_proxy/collision/Proxy_V1_collision.STL" scale="0.001 0.001 0.001"/>-->
+        </geometry>
+      </collision>
+    </link>
+    <link name="apple" >
+      <visual>
+        <origin xyz="0 0 0" rpy="0 0 0"/>
+        <geometry>
+          <mesh filename="package://millrace_moveit_config/meshes/apple_proxy/visual/SubAssem_Apple_V4.STL" scale="0.001 0.001 0.001"/>
+        </geometry>
+        <material name="Red">
+          <color rgba="1.0 0.0 0.0 1.0"/>
+        </material>
+      </visual>
+    </link>
   </xacro:macro>
 </robot>

File: urdf/ur5e.xacro (robot description, xacro)
@@ -17,10 +17,10 @@
   <xacro:include filename="$(find ur_description)/urdf/inc/ur5e_macro.xacro"/>
   <xacro:ur5e_robot prefix=""/>
+  <!-- In addition to the above, we would also like to define a table and some more joints -->
+  <link name="world" />
+  <link name="palm" />
   <!--  Tables and Walls -->
   <xacro:include filename="$(find millrace_moveit_config)/urdf/tables_v2.urdf.xacro" />
   <xacro:tables />
-  <!-- In addition to the above, we would also like to define a table and some more joints -->
-  <link name="world" />
-  <link name="palm" />
   <!-- Describe the interface between the robot and the gripper -->
   <joint name="robotiq_coupler_joint" type="fixed">
@@ -59,3 +59,15 @@
     <origin xyz="0 0 0.165" rpy="0 0 0.2618 " />      <!-- Add in Z the hand's thickness (approx 13cm) -->
   </joint>
+  <joint name = "proxy_stem" type="fixed">
+    <parent link = "apple_proxy" />
+    <child link = "apple_stem" />
+    <!-- <origin xyz = "0.16 0.45 2.42" rpy="0 3.1416 0.0" /> -->
+    <origin xyz = "0.3 0.25 0.25" rpy="1.5708 0 0" />
+  </joint>
+  <joint name = "stem_apple" type="fixed">
+    <parent link = "apple_stem" />
+    <child link = "apple" />
+    <!-- <origin xyz = "-0.04 -0.03 -2.08" rpy="0 0.0 0.0" /> -->
+    <origin xyz = "-0.04 -0.03 0.03" rpy="0 0 0" />
+  </joint>
 </robot>

Commit message: scene and workspace updates

File: urdf/tables_v2.urdf.xacro (robot description, xacro)
@@ -54,5 +54,5 @@
     </link>
     <!-- Simplified Version of Lisa's hand -->
-    <link name="lisas_hand">
+    <!-- <link name="lisas_hand">
       <visual>
         <origin xyz="0 0 0" rpy="0 0 0"/>
@@ -70,8 +70,9 @@
         </geometry>
       </collision>
-    </link>
+    </link> -->
     <link name="apple_stem" >
       <visual>
-        <origin xyz="0 0 0" rpy="0 0 0"/>
+        <!-- <origin xyz="0 0 0" rpy="0 0 0"/> -->
+        <origin xyz="-.0095851 -.0115 0" rpy="0 0 0"/>
         <geometry>
           <mesh filename="package://millrace_moveit_config/meshes/apple_proxy/visual/Stem_v4.STL" scale="0.001 0.001 0.001"/>
@@ -82,5 +83,6 @@
       </visual>
       <collision>
-        <origin xyz="0 0 0" rpy="0 0 0"/>
+        <!-- <origin xyz="0 0 0" rpy="0 0 0"/> -->
+        <origin xyz="-.0095851 0 0" rpy="0 0 0"/>
         <geometry>
           <mesh filename="package://millrace_moveit_config/meshes/apple_proxy/collision/Proxy_V1_collision.STL" scale="0.001 0.001 0.001"/>-->
@@ -90,5 +92,6 @@
     <link name="apple" >
       <visual>
-        <origin xyz="0 0 0" rpy="0 0 0"/>
+        <!-- <origin xyz="0 0 0" rpy="0 0 0"/> -->
+        <origin xyz="-.0417815 -.0417815 -.0418201" rpy="0 0 0"/>
         <geometry>
           <mesh filename="package://millrace_moveit_config/meshes/apple_proxy/visual/SubAssem_Apple_V4.STL" scale="0.001 0.001 0.001"/>

File: urdf/ur5e.xacro (robot description, xacro)
@@ -24,9 +24,9 @@
   <xacro:tables />
   <!-- Describe the interface between the robot and the gripper -->
-  <joint name="robotiq_coupler_joint" type="fixed">
+  <!-- <joint name="robotiq_coupler_joint" type="fixed">
     <parent link="tool0" />
     <child link="lisas_hand" />
     <origin xyz="-0.0675 0.0675 0.004" rpy="0 0 ${-pi/2.0}" />
-  </joint>
+  </joint> -->
   <!-- Describe the interface between the world and the tables -->
   <joint name="world_big_table" type="fixed">
@@ -56,6 +56,7 @@
     <parent link="tool0" />
     <child link="palm" />
-  <!--    <origin xyz="0 0 0.13" rpy="0 0 0.2618 " />      &lt;!&ndash; Add in Z the hand's thickness (approx 13cm) &ndash;&gt;-->
-    <origin xyz="0 0 0.165" rpy="0 0 0.2618 " />      <!-- Add in Z the hand's thickness (approx 13cm) -->
+    <!--    <origin xyz="0 0 0.13" rpy="0 0 0.2618 " />      &lt;!&ndash; Add in Z the hand's thickness (approx 13cm) &ndash;&gt;-->
+    <!--  <origin xyz="0 0 0.165" rpy="0 0 0.2618 " /> -->     <!-- Add in Z the hand's thickness (approx 13cm) -->
+    <origin xyz="0 0 0.1" rpy="0 0 0 " />     <!-- Add in Z the hand's thickness (approx 10cm) -->
   </joint>
   <joint name = "proxy_stem" type="fixed">
@@ -69,5 +70,5 @@
     <child link = "apple" />
     <!-- <origin xyz = "-0.04 -0.03 -2.08" rpy="0 0.0 0.0" /> -->
-    <origin xyz = "-0.04 -0.03 0.03" rpy="0 0 0" />
+    <origin xyz = "0 0 0.07" rpy="0 0 0" />
   </joint>
 </robot>

Commit message: fix: remove stem collision and reposition apple

File: urdf/tables_v2.urdf.xacro (robot description, xacro)
@@ -82,11 +82,11 @@
         </material>
       </visual>
-      <collision>
-        <!-- <origin xyz="0 0 0" rpy="0 0 0"/> -->
+      <!-- <collision>
+        <!- <origin xyz="0 0 0" rpy="0 0 0"/> ->
         <origin xyz="-.0095851 0 0" rpy="0 0 0"/>
         <geometry>
-          <mesh filename="package://millrace_moveit_config/meshes/apple_proxy/collision/Proxy_V1_collision.STL" scale="0.001 0.001 0.001"/>-->
+          <mesh filename="package://millrace_moveit_config/meshes/apple_proxy/collision/Proxy_V1_collision.STL" scale="0.001 0.001 0.001"/>
         </geometry>
-      </collision>
+      </collision> -->
     </link>
     <link name="apple" >

File: urdf/ur5e.xacro (robot description, xacro)
@@ -64,5 +64,5 @@
     <child link = "apple_stem" />
     <!-- <origin xyz = "0.16 0.45 2.42" rpy="0 3.1416 0.0" /> -->
-    <origin xyz = "0.3 0.25 0.25" rpy="1.5708 0 0" />
+    <origin xyz = "0.2 0.25 0.25" rpy="1.5708 0 0" />
   </joint>
   <joint name = "stem_apple" type="fixed">

Commit message: fix: move install to rospkg, rename repository

File: urdf/tables_v2.urdf.xacro (robot description, xacro)
@@ -6,5 +6,5 @@
         <origin xyz="0 0 0" rpy="0 0 0"/>
         <geometry>
-          <mesh filename="package://millrace_moveit_config/meshes/furniture/collision/UR5_big_table.STL" scale="0.001 0.001 0.001"/>
+          <mesh filename="package://applevision_moveit_config/meshes/furniture/collision/UR5_big_table.STL" scale="0.001 0.001 0.001"/>
         </geometry>
         <material name="Grey">
@@ -15,5 +15,5 @@
         <origin xyz="0 0 0" rpy="0 0 0"/>
         <geometry>
-          <mesh filename="package://millrace_moveit_config/meshes/furniture/collision/UR5_big_table.STL" scale="0.001 0.001 0.001"/>
+          <mesh filename="package://applevision_moveit_config/meshes/furniture/collision/UR5_big_table.STL" scale="0.001 0.001 0.001"/>
         </geometry>
       </collision>
@@ -23,5 +23,5 @@
         <origin xyz="0 0 0" rpy="0 0 0"/>
         <geometry>
-          <mesh filename="package://millrace_moveit_config/meshes/furniture/collision/UR5_small_table.STL" scale="0.001 0.001 0.001"/>
+          <mesh filename="package://applevision_moveit_config/meshes/furniture/collision/UR5_small_table.STL" scale="0.001 0.001 0.001"/>
         </geometry>
         <material name="Grey">
@@ -32,5 +32,5 @@
         <origin xyz="0 0 0" rpy="0 0 0"/>
         <geometry>
-          <mesh filename="package://millrace_moveit_config/meshes/furniture/collision/UR5_small_table.STL" scale="0.001 0.001 0.001"/>
+          <mesh filename="package://applevision_moveit_config/meshes/furniture/collision/UR5_small_table.STL" scale="0.001 0.001 0.001"/>
         </geometry>
       </collision>
@@ -40,5 +40,5 @@
         <origin xyz="0 0 0" rpy="0 0 0"/>
         <geometry>
-          <mesh filename="package://millrace_moveit_config/meshes/furniture/collision/UR5_simpleProxy.STL" scale="0.001 0.001 0.001"/>
+          <mesh filename="package://applevision_moveit_config/meshes/furniture/collision/UR5_simpleProxy.STL" scale="0.001 0.001 0.001"/>
         </geometry>
         <material name="Green">
@@ -49,5 +49,5 @@
         <origin xyz="0 0 0" rpy="0 0 0"/>
         <geometry>
-          <mesh filename="package://millrace_moveit_config/meshes/furniture/collision/UR5_simpleProxy.STL" scale="0.001 0.001 0.001"/>
+          <mesh filename="package://applevision_moveit_config/meshes/furniture/collision/UR5_simpleProxy.STL" scale="0.001 0.001 0.001"/>
         </geometry>
       </collision>
@@ -58,5 +58,5 @@
         <origin xyz="0 0 0" rpy="0 0 0"/>
         <geometry>
-          <mesh filename="package://millrace_moveit_config/meshes/hand/hand_cylinder.STL" scale="0.001 0.001 0.001"/>
+          <mesh filename="package://applevision_moveit_config/meshes/hand/hand_cylinder.STL" scale="0.001 0.001 0.001"/>
         </geometry>
         <material name="Black">
@@ -67,5 +67,5 @@
         <origin xyz="0 0 0" rpy="0 0 0"/>
         <geometry>
-          <mesh filename="package://millrace_moveit_config/meshes/hand/hand_cylinder.STL" scale="0.001 0.001 0.001"/>
+          <mesh filename="package://applevision_moveit_config/meshes/hand/hand_cylinder.STL" scale="0.001 0.001 0.001"/>
         </geometry>
       </collision>
@@ -76,5 +76,5 @@
         <origin xyz="-.0095851 -.0115 0" rpy="0 0 0"/>
         <geometry>
-          <mesh filename="package://millrace_moveit_config/meshes/apple_proxy/visual/Stem_v4.STL" scale="0.001 0.001 0.001"/>
+          <mesh filename="package://applevision_moveit_config/meshes/apple_proxy/visual/Stem_v4.STL" scale="0.001 0.001 0.001"/>
         </geometry>
         <material name="Orange">
@@ -86,5 +86,5 @@
         <origin xyz="-.0095851 0 0" rpy="0 0 0"/>
         <geometry>
-          <mesh filename="package://millrace_moveit_config/meshes/apple_proxy/collision/Proxy_V1_collision.STL" scale="0.001 0.001 0.001"/>
+          <mesh filename="package://applevision_moveit_config/meshes/apple_proxy/collision/Proxy_V1_collision.STL" scale="0.001 0.001 0.001"/>
         </geometry>
       </collision> -->
@@ -95,5 +95,5 @@
         <origin xyz="-.0417815 -.0417815 -.0418201" rpy="0 0 0"/>
         <geometry>
-          <mesh filename="package://millrace_moveit_config/meshes/apple_proxy/visual/SubAssem_Apple_V4.STL" scale="0.001 0.001 0.001"/>
+          <mesh filename="package://applevision_moveit_config/meshes/apple_proxy/visual/SubAssem_Apple_V4.STL" scale="0.001 0.001 0.001"/>
         </geometry>
         <material name="Red">

File: urdf/ur5e.xacro (robot description, xacro)
@@ -21,5 +21,5 @@
   <link name="palm" />
   <!--  Tables and Walls -->
-  <xacro:include filename="$(find millrace_moveit_config)/urdf/tables_v2.urdf.xacro" />
+  <xacro:include filename="$(find applevision_moveit_config)/urdf/tables_v2.urdf.xacro" />
   <xacro:tables />
   <!-- Describe the interface between the robot and the gripper -->

Commit message: updating xacro measurements

File: urdf/tables_v2.urdf.xacro (robot description, xacro)
@@ -40,5 +40,5 @@
         <origin xyz="0 0 0" rpy="0 0 0"/>
         <geometry>
-          <mesh filename="package://apple_proxy/meshes/apple_proxy/collision/apple_proxy_collision.STL" scale="0.001 0.001 0.001"/>
+          <mesh filename="package://applevision_moveit_config/meshes/apple_proxy/visual/apple_proxy_visual.STL" scale="0.001 0.001 0.001"/>
         </geometry>
         <material name="Green">
@@ -49,14 +49,14 @@
         <origin xyz="0 0 0" rpy="0 0 0"/>
         <geometry>
-          <mesh filename="package://apple_proxy/meshes/apple_proxy/collision/apple_proxy_collision.STL" scale="0.001 0.001 0.001"/>
+          <mesh filename="package://applevision_moveit_config/meshes/apple_proxy/collision/apple_proxy_collision.STL" scale="0.001 0.001 0.001"/>
         </geometry>
       </collision>
     </link>
     <!-- Simplified Version of Lisa's hand -->
-    <!-- <link name="lisas_hand">
+    <link name="lisas_hand">
       <visual>
         <origin xyz="0 0 0" rpy="0 0 0"/>
         <geometry>
-          <mesh filename="package://applevision_moveit_config/meshes/hand/hand_cylinder.STL" scale="0.001 0.001 0.001"/>
+          <mesh filename="package://applevision_moveit_config/meshes/hand/hand_cylinder.STL" scale="0.001 0.001 0.0012"/>
         </geometry>
         <material name="Black">
@@ -70,5 +70,5 @@
         </geometry>
       </collision>
-    </link> -->
+    </link>
     <link name="apple_stem" >
       <visual>

File: urdf/ur5e.xacro (robot description, xacro)
@@ -24,9 +24,9 @@
   <link name="palm" />
   <!-- Describe the interface between the robot and the gripper -->
-  <!-- <joint name="robotiq_coupler_joint" type="fixed">
+  <joint name="robotiq_coupler_joint" type="fixed">
     <parent link="tool0" />
     <child link="lisas_hand" />
     <origin xyz="-0.0675 0.0675 0.004" rpy="0 0 ${-pi/2.0}" />
-  </joint> -->
+  </joint>
   <!-- Describe the interface between the world and the tables -->
   <joint name="world_big_table" type="fixed">
@@ -38,5 +38,5 @@
     <parent link="world" />
     <child link="small_table" />
-    <origin xyz="-0.21 -1.37 0" rpy="0 0 1.5708" />
+    <origin xyz="-0.21 -1.40 0" rpy="0 0 1.5708" />
   </joint>
   <!-- Describe the interface between the world and the Apple Proxy -->
@@ -44,5 +44,5 @@
     <parent link = "big_table" /> -->
     <child link = "apple_proxy" /> -->
-    <origin xyz = ".48 .8 .95" rpy="1.5708 0 -1.5708" />
+    <origin xyz = ".462 1.027 1.672" rpy="3.1416 1.5708 0" />
   </joint>
   <!-- Describe the interface between the world and the robot" -->
@@ -50,5 +50,5 @@
     <parent link="small_table" />
     <child link = "base_link" />
-    <origin xyz="0.355 0.357 0.86" rpy="0.0 0.0 3.1416" />
+    <origin xyz="0.272 0.357 0.858" rpy="0.0 0.0 3.1416" />
   </joint>
   <!-- Describe the location of the palm -->
@@ -57,5 +57,5 @@
     <child link="palm" />
 <!--        <origin xyz="0 0 0.13" rpy="0 0 0.2618 " />      &lt;!&ndash; Add in Z the hand's thickness (approx 13cm) &ndash;&gt;-->
-    <origin xyz="0 0 0" rpy="0 0 0.2618 " />      <!-- Add in Z the hand's thickness (approx 13cm) -->
+    <origin xyz="0 0 .165" rpy="0 0 -.7 " />      <!-- Add in Z the hand's thickness (approx 13cm) -->
   </joint>
   <!-- <joint name = "apple_proxy" type = "fixed">
@@ -76,5 +76,5 @@
     <child link = "apple" />
     <!-- <origin xyz = "-0.04 -0.03 -2.08" rpy="0 0.0 0.0" /> -->
-    <origin xyz = "0 0 0.07" rpy="0 0 0" />
+    <origin xyz = "0 0 .095" rpy="0 0 0" />
   </joint>
 </robot>
