Commit message: fix: minor urdf updates

File: urdf/ur5e.xacro (robot description, xacro)
@@ -58,5 +58,5 @@
     <!--    <origin xyz="0 0 0.13" rpy="0 0 0.2618 " />      &lt;!&ndash; Add in Z the hand's thickness (approx 13cm) &ndash;&gt;-->
     <!--  <origin xyz="0 0 0.165" rpy="0 0 0.2618 " /> -->     <!-- Add in Z the hand's thickness (approx 13cm) -->
-    <origin xyz="0 0 0.1" rpy="0 0 0 " />     <!-- Add in Z the hand's thickness (approx 10cm) -->
+    <origin xyz="0 0 0.05" rpy="0 0 0.2618 "/>     <!-- Add in Z the hand's thickness (approx 5cm) -->
   </joint>
   <joint name = "proxy_stem" type="fixed">

Commit message: feat: millrace changes

File: urdf/ur5e.xacro (robot description, xacro)
@@ -33,5 +33,5 @@
     <parent link="world" />
     <child link="big_table" />
-    <origin xyz="0 0 0" rpy="0 0 1.5708" />
+    <origin xyz="0 0 0.145" rpy="0 0 1.5708" />
   </joint>
   <joint name="world_small_table" type="fixed">
@@ -58,5 +58,5 @@
     <!--    <origin xyz="0 0 0.13" rpy="0 0 0.2618 " />      &lt;!&ndash; Add in Z the hand's thickness (approx 13cm) &ndash;&gt;-->
     <!--  <origin xyz="0 0 0.165" rpy="0 0 0.2618 " /> -->     <!-- Add in Z the hand's thickness (approx 13cm) -->
-    <origin xyz="0 0 0.05" rpy="0 0 0.2618 "/>     <!-- Add in Z the hand's thickness (approx 5cm) -->
+    <origin xyz="0 0 0.05" rpy="0 0 5.55"/>     <!-- Add in Z the hand's thickness (approx 5cm) -->
   </joint>
   <joint name = "proxy_stem" type="fixed">
@@ -64,5 +64,5 @@
     <child link = "apple_stem" />
     <!-- <origin xyz = "0.16 0.45 2.42" rpy="0 3.1416 0.0" /> -->
-    <origin xyz = "0.2 0.25 0.25" rpy="1.5708 0 0" />
+    <origin xyz = "0.3 0.25 0.25" rpy="1.5708 0 0" />
   </joint>
   <joint name = "stem_apple" type="fixed">

Commit message: trying to find what went wrong

File: urdf/ur5e.xacro (robot description, xacro)
@@ -33,10 +33,10 @@
     <parent link="world" />
     <child link="big_table" />
-    <origin xyz="-.01 0 0.145" rpy="0 0 1.5708" />
+    <origin xyz="-.01 0 0" rpy="0 0 1.5708" />
   </joint>
   <joint name="world_small_table" type="fixed">
     <parent link="world" />
     <child link="small_table" />
-    <origin xyz="-0.21 -1.40 0" rpy="0 0 1.5708" />
+    <origin xyz="-0.21 -1.535 0" rpy="0 0 1.5708" />
   </joint>
   <!-- Describe the interface between the world and the Apple Proxy -->
@@ -44,5 +44,5 @@
     <parent link = "big_table" /> -->
     <child link = "apple_proxy" /> -->
-    <origin xyz = ".462 1.027 1.672" rpy="3.1416 1.5708 0" />
+    <origin xyz = ".462 1.027 1.67" rpy="3.1416 1.5708 0" />
   </joint>
   <!-- Describe the interface between the world and the robot" -->
@@ -53,9 +53,10 @@
   </joint>
   <!-- Describe the location of the palm -->
+  FIX THIS AHHHHHHHHH
   <joint name="hand_palm" type="fixed">
     <parent link="tool0" />
     <child link="palm" />
 <!--        <origin xyz="0 0 0.13" rpy="0 0 0.2618 " />      &lt;!&ndash; Add in Z the hand's thickness (approx 13cm) &ndash;&gt;-->
-    <origin xyz="0 0 .165" rpy="0 0 -.7 " />      <!-- Add in Z the hand's thickness (approx 13cm) -->
+    <origin xyz="0 0 .165" rpy="0 0 -1.57 " />      <!-- Add in Z the hand's thickness (approx 13cm) -->
   </joint>
   <!-- <joint name = "apple_proxy" type = "fixed">
@@ -66,15 +67,15 @@
   <!--</joint> -->
   <joint name = "proxy_stem" type="fixed">
-    <parent link = "apple_proxy" />
+    <parent link = "base_link" />
     <child link = "apple_stem" />
     <!-- <origin xyz = "0.16 0.45 2.42" rpy="0 3.1416 0.0" /> -->
     <!-- <origin xyz = "0 0 -.05" rpy="1.5708 0 0" /> -->
-    <origin xyz = ".225 .35 .73" rpy="1.5708 0 0" />
+    <origin xyz = "-.99 -.1205 .5525" rpy="1.5708 0 0" />
   </joint>
   <joint name = "stem_apple" type="fixed">
-    <parent link = "apple_stem" />
+    <parent link = "base_link" />
     <child link = "apple" />
     <!-- <origin xyz = "-0.04 -0.03 -2.08" rpy="0 0.0 0.0" /> -->
-    <origin xyz = "0 0 .095" rpy="0 0 0" />
+    <origin xyz = "-.99 -.1205 .5225" rpy="0 0 0" />
   </joint>
 </robot>

Commit message: debuggin

File: urdf/ur5e.xacro (robot description, xacro)
@@ -58,5 +58,5 @@
     <child link="palm" />
 <!--        <origin xyz="0 0 0.13" rpy="0 0 0.2618 " />      &lt;!&ndash; Add in Z the hand's thickness (approx 13cm) &ndash;&gt;-->
-    <origin xyz="0 0 .165" rpy="0 0 -1.57 " />      <!-- Add in Z the hand's thickness (approx 13cm) -->
+    <origin xyz="0 0 .165" rpy="0 0 2.44346" />      <!-- Add in Z the hand's thickness (approx 13cm) (with new hand: yaw is -1.57)-->
   </joint>
   <!-- <joint name = "apple_proxy" type = "fixed">

Commit message: working again(?)

File: urdf/ur5e.xacro (robot description, xacro)
@@ -53,10 +53,9 @@
   </joint>
   <!-- Describe the location of the palm -->
-  FIX THIS AHHHHHHHHH
   <joint name="hand_palm" type="fixed">
     <parent link="tool0" />
     <child link="palm" />
 <!--        <origin xyz="0 0 0.13" rpy="0 0 0.2618 " />      &lt;!&ndash; Add in Z the hand's thickness (approx 13cm) &ndash;&gt;-->
-    <origin xyz="0 0 .165" rpy="0 0 2.44346" />      <!-- Add in Z the hand's thickness (approx 13cm) (with new hand: yaw is -1.57)-->
+    <origin xyz="0 0 .165" rpy="0 0 -.706" />      <!-- Add in Z the hand's thickness (approx 13cm) (with new hand: yaw is -1.57)-->
   </joint>
   <!-- <joint name = "apple_proxy" type = "fixed">
